File: Full555Timer/Full555Timer.kicad_pcb (KiCad board)
At the start: 4 copper layers, 130.2 x 64.1 mm, 51 parts, among them J1 GND, J2 5V, J3 HLT, J4 /CLK, J5 CLK, J6 HLTGND, J7 HLT5V, SW1 SWITCH, SW2 SPDT, U1 NE555P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

Commit message: Add files via upload
Parts:
- removed *: *, Full555Timer:test5
- U1: value NE555P -> NE555
- U2, U3: value LM555CN -> NE555
- moved D4 1.80 mm to (203.2, 104.1), turned to -90 degrees
Routing:
- net Net-(D4-Pad1): track 26.5 -> 28.2 mm
- net Net-(D4-Pad2): track 46.0 -> 47.8 mm
- net Net-(U4-Pad10): track 62.7 -> 62.1 mm
- net +5V: track 368.8 -> 368.2 mm
- net GND: track 398.4 -> 397.7 mm
Other:
- net class Default removed
- board text added: "555 Timer Board v0.1 1/9/2022 Toberdyne/Tom Whitson"
- board text removed: "555 Timer Board v1 10/4/20 Toberdyne Industries"
