File: Full555Timer/Full555Timer.sch (KiCad schematic (older format))
At the start: 50 parts, among them J1 GND, J2 5V, J3 HLT, J4 /CLK, J5 CLK, J6 HLTGND, J7 HLT5V, SW1 SWITCH, SW2 SPDT, U1 NE555P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

Commit message: Add files via upload
Connections:
- net at C3.1, RV1.1, U1.2 (TR)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: now also D1.2 (A), U4.1
- now unconnected: U1.3 (Q)
